File: PCB/kicad/power.kicad_sch (KiCad schematic)
At the start: 54 parts, among them J1 12V HEAT IN, J2 12V MAIN IN, J3 USB-C 5V OUT, Q11 AO3401A, Q12 AO3401A, U1 LMR33630ADDA, U11 TLV7041, U2 AP2112K-3.3

Commit message: new board
Parts:
- removed C11: 1uF 16V, Capacitor_SMD:C_0603_1608Metric, symbol Device:C
- removed C12: 2.2uF 16V, Capacitor_SMD:C_0603_1608Metric, symbol Device:C
- removed C2: 10uF 50V, Capacitor_SMD:C_1210_3225Metric, symbol Device:C
- removed C65: 100nF, Capacitor_SMD:C_0603_1608Metric, symbol Device:C
- removed D45, D46: 1N4148WS, Diode_SMD:D_SOD-323, symbol Diode:1N4148WS
- removed H3: M3, MountingHole:MountingHole_3.2mm_M3, symbol Mechanical:MountingHole
- removed J3: USB-C 5V OUT, Connector_USB:USB_C_Receptacle_GCT_USB4125-xx-x_6P_TopMnt_Horizontal, symbol Connector:USB_C_Receptacle_PowerOnly_6P
- removed Q11, Q12: AO3401A, Package_TO_SOT_SMD:SOT-23, symbol Transistor_FET:AO3401A
- removed R89, R90: 56k, Resistor_SMD:R_0603_1608Metric, symbol Device:R
- removed R91: 220k, Resistor_SMD:R_0603_1608Metric, symbol Device:R
- removed R92, R96: 10k, Resistor_SMD:R_0603_1608Metric, symbol Device:R
- removed R94, R95: 100k, Resistor_SMD:R_0603_1608Metric, symbol Device:R
- removed U11: TLV7041, Package_TO_SOT_SMD:SOT-23-5, symbol Comparator:TLV7041DBV
- added F8: 2A, Fuse:Fuse_1812_4532Metric, symbol Device:Polyfuse
- added J28: 12V OUT, FM:TB_DB301V-3.5-2P, symbol Connector_Generic:Conn_01x02
- added J29: 5V OUT, FM:TB_DB301V-3.5-2P, symbol Connector_Generic:Conn_01x02
- added U1: LMR33630ADDA, Package_SO:TI_SO-PowerPAD-8_ThermalVias, symbol Regulator_Switching:LMR33630ADDA
- C1: renamed from U1; value LMR33630ADDA -> 100uF 35V; footprint Package_SO:TI_SO-PowerPAD-8_ThermalVias -> Capacitor_THT:CP_Radial_D6.3mm_P2.50mm; symbol Regulator_Switching:LMR33630ADDA -> Device:C_Polarized; LCSC (none) -> C106694; MPN LMR33630ADDAR -> ERS1VM101E12OT; Manufacturer Texas Instruments -> AISHI
- C10: renamed from U2; value AP2112K-3.3 -> 22uF 25V; footprint Package_TO_SOT_SMD:SOT-23-5 -> Capacitor_SMD:C_1206_3216Metric; symbol Regulator_Linear:AP2112K-3.3 -> Device:C; LCSC (none) -> C12891; MPN AP2112K-3.3TRG1 -> MLCC 22uF 25V; Manufacturer Diodes Inc. -> Samsung/Yageo (JLCPCB basic)
- C2: renamed from C3; footprint Capacitor_SMD:C_1210_3225Metric -> Capacitor_SMD:C_1206_3216Metric; LCSC (none) -> C13585; MPN GRM32ER71H106KA12L -> MLCC 10uF 50V; Manufacturer Samsung/Murata (generic) -> Samsung/Yageo (JLCPCB basic)
- C3: renamed from C4; value 220nF 50V -> 10uF 50V; footprint Capacitor_SMD:C_0603_1608Metric -> Capacitor_SMD:C_1206_3216Metric; LCSC (none) -> C13585; MPN CL10B224KB8NNNC -> MLCC 10uF 50V; Manufacturer Samsung/Murata (generic) -> Samsung/Yageo (JLCPCB basic)
- C4: renamed from C5; value 100nF -> 220nF 50V; footprint Capacitor_SMD:C_0603_1608Metric -> Capacitor_SMD:C_0805_2012Metric; LCSC (none) -> C5378; MPN MLCC 100nF -> MLCC 220nF 50V; Manufacturer Samsung/Murata (generic) -> Samsung/Yageo (JLCPCB basic)
- C5: renamed from C6; value 1uF 16V -> 100nF; LCSC (none) -> C14663; MPN MLCC 1uF 16V -> MLCC 100nF; Manufacturer Samsung/Murata (generic) -> Samsung/Yageo (JLCPCB basic)
- C6: renamed from L1; value 6.8uH -> 1uF 50V; footprint Inductor_SMD:L_Bourns_SRP7028A_7.3x6.6mm -> Capacitor_SMD:C_0603_1608Metric; symbol Device:L -> Device:C; LCSC (none) -> C15849; MPN SRP7028A-6R8M -> MLCC 1uF 50V; Manufacturer Bourns -> Samsung/Yageo (JLCPCB basic)
- C63: value 4.7uF 16V -> 10uF 25V; LCSC (none) -> C15850; MPN MLCC 4.7uF 16V -> MLCC 10uF 25V; Manufacturer Samsung/Murata (generic) -> Samsung/Yageo (JLCPCB basic)
- C64: value 100nF -> 10uF 25V; footprint Capacitor_SMD:C_0603_1608Metric -> Capacitor_SMD:C_0805_2012Metric; LCSC (none) -> C15850; MPN MLCC 100nF -> MLCC 10uF 25V; Manufacturer Samsung/Murata (generic) -> Samsung/Yageo (JLCPCB basic)
- C7: renamed from C8; value 22uF 16V -> 22uF 25V; LCSC (none) -> C12891; MPN CL31A226KOHNNNE -> MLCC 22uF 25V; Manufacturer Samsung/Murata (generic) -> Samsung/Yageo (JLCPCB basic)
- C8: renamed from C9; value 22uF 16V -> 22uF 25V; LCSC (none) -> C12891; MPN CL31A226KOHNNNE -> MLCC 22uF 25V; Manufacturer Samsung/Murata (generic) -> Samsung/Yageo (JLCPCB basic)
- C9: renamed from C10; value 22uF 16V -> 22uF 25V; LCSC (none) -> C12891; MPN CL31A226KOHNNNE -> MLCC 22uF 25V; Manufacturer Samsung/Murata (generic) -> Samsung/Yageo (JLCPCB basic)
- D1: renamed from D2; value SMCJ16A -> SMBJ16A; footprint Diode_SMD:D_SMC -> Diode_SMD:D_SMB; LCSC (none) -> C19077571; MPN SMCJ16A -> SMBJ16A; Manufacturer Littelfuse -> hongjiacheng
- D2: renamed from C1; value 100uF 25V -> SMBJ16A; footprint Capacitor_THT:CP_Radial_D8.0mm_P3.50mm -> Diode_SMD:D_SMB; symbol Device:C_Polarized -> Device:D_Zener; LCSC (none) -> C19077571; MPN EEU-FR1E101 -> SMBJ16A; Manufacturer Panasonic -> hongjiacheng
- D3, D4, D5: footprint LED_SMD:LED_0603_1608Metric -> LED_SMD:LED_0805_2012Metric; LCSC (none) -> C2297; MPN KT-0603G -> KT-0805G
- F1: renamed from F2; value 15A MINI -> 15A; footprint Fuse:Fuseholder_Blade_Mini_Keystone_3568 -> FM:FUSE_2410_SMD; LCSC (none) -> C136393; MPN 3568 -> JFC2410-2150TS; Manufacturer Keystone -> Shenzhen JDT Fuse
- F2: renamed from F3; value 15A MINI -> 15A; footprint Fuse:Fuseholder_Blade_Mini_Keystone_3568 -> FM:FUSE_2410_SMD; LCSC (none) -> C136393; MPN 3568 -> JFC2410-2150TS; Manufacturer Keystone -> Shenzhen JDT Fuse
- F3: renamed from F4; value 7.5A MINI -> 15A; footprint Fuse:Fuseholder_Blade_Mini_Keystone_3568 -> FM:FUSE_2410_SMD; LCSC (none) -> C136393; MPN 3568 -> JFC2410-2150TS; Manufacturer Keystone -> Shenzhen JDT Fuse
- F4: renamed from D1; value SMCJ16A -> 8A; footprint Diode_SMD:D_SMC -> FM:FUSE_2410_SMD; symbol Device:D_Zener -> Device:Fuse; LCSC (none) -> C136390; MPN SMCJ16A -> JFC2410-1800TS; Manufacturer Littelfuse -> Shenzhen JDT Fuse
- F5: value 1.5A -> 1.1A; LCSC (none) -> C269134; MPN 1812L150/12DR -> SMD1812B110TF/33; Manufacturer Littelfuse -> Brightking
- F6: LCSC (none) -> C720075; MPN 1206L050YR -> JK-nSMD050-30; Manufacturer Littelfuse -> Jinrui
- H3: renamed from R93; value 130k -> M3; footprint Resistor_SMD:R_0603_1608Metric -> MountingHole:MountingHole_3.2mm_M3; symbol Device:R -> Mechanical:MountingHole; MPN 0603 130k 1% -> (none); Manufacturer Yageo/UniOhm (generic) -> (none); now left out of the parts list
- J1: value 12V HEAT IN -> 12V IN HEATER 1; footprint TerminalBlock_Phoenix:TerminalBlock_Phoenix_MKDS-3-2-5.08_1x02_P5.08mm_Horizontal -> FM:TB_WJ500V-5.08-2P; LCSC (none) -> C8465; MPN 1711026 -> WJ500V-5.08-2P; Manufacturer Phoenix Contact -> Ningbo Kangnex
- J2: value 12V MAIN IN -> 12V IN HEATER 2; footprint TerminalBlock_Phoenix:TerminalBlock_Phoenix_MKDS-3-2-5.08_1x02_P5.08mm_Horizontal -> FM:TB_WJ500V-5.08-2P; LCSC (none) -> C8465; MPN 1711026 -> WJ500V-5.08-2P; Manufacturer Phoenix Contact -> Ningbo Kangnex
- J3: renamed from F1; value 15A MINI -> 12V IN MAIN; footprint Fuse:Fuseholder_Blade_Mini_Keystone_3568 -> FM:TB_WJ500V-5.08-2P; symbol Device:Fuse -> Connector_Generic:Conn_01x02; LCSC (none) -> C8465; MPN 3568 -> WJ500V-5.08-2P; Manufacturer Keystone -> Ningbo Kangnex
- L1: renamed from R1; value 100k -> 10uH; footprint Resistor_SMD:R_0603_1608Metric -> FM:L_SLO0630H; symbol Device:R -> Device:L; LCSC (none) -> C207842; MPN 0603 100k 1% -> SLO0630H100MTT; Manufacturer Yageo/UniOhm (generic) -> Sunltech
- R1: renamed from R2; value 24.3k -> 100k; LCSC (none) -> C25803; MPN 0603 24.3k 1% -> 0603 100k 1%; Manufacturer Yageo/UniOhm (generic) -> UNI-ROYAL
- R2: renamed from C7; value 22uF 16V -> 24k; footprint Capacitor_SMD:C_1206_3216Metric -> Resistor_SMD:R_0603_1608Metric; symbol Device:C -> Device:R; LCSC (none) -> C23352; MPN CL31A226KOHNNNE -> 0603 24k 1%; Manufacturer Samsung/Murata (generic) -> UNI-ROYAL
- R3: LCSC (none) -> C23162; Manufacturer Yageo/UniOhm (generic) -> UNI-ROYAL
- R4, R5: LCSC (none) -> C21190; Manufacturer Yageo/UniOhm (generic) -> UNI-ROYAL
Connections:
- net USBC_GATE is gone; now on net +5V_AUX: C64.1
- net +12V: now also C1.1, C4.1, D1.1 (K), F4.2, F8.1, U1.2 (VIN), U1.3 (EN); no longer C1.2 (VIN), C1.3 (EN), D2.1, F3.2, F4.1 (K)
- net +12V_H1: now also F1.2; no longer J3.2
- net +12V_H2: now also F2.2; no longer F1.2
- net +12V_IN_M: now also F4.1, J3.2 (Pin_2); no longer F2.1, J2.2 (Pin_2)
- net +12V_PUMP: now also D2.1 (K), F3.2; no longer D1.1 (K), F2.2
- net +3V3: no longer C10.5 (VOUT)
- net +5V: now also L1.2, R1.1; no longer C10.3 (EN), C6.2, L1.1, R2.1
- net BUCK_BOOT: now also C5.1, U1.7 (BOOT); no longer C1.7 (BOOT), C4.1
- net BUCK_FB: now also R1.2, R2.1, U1.5 (FB); no longer C1.5 (FB), L1.2, R1.1
- net BUCK_SW: now also C5.2, L1.1, U1.8 (SW); no longer C1.8 (SW), C4.2, C6.1
- net BUCK_VCC: now also C6.1, U1.6 (VCC); no longer C1.6 (VCC), C5.1
- net GND: now also C1.2, C4.2, C6.2, C64.2, J3.1 (Pin_1), J28.1 (Pin_1), J29.1 (Pin_1), U1.1 (GND), U1.9 (GND); no longer C1.1 (GND), C1.9 (GND), C5.2, F4.2 (A), R1.2
- net +12V_IN_H renamed +12V_IN_H1
- net +12V_IN_H1: no longer J3.1
- net +5V_USB renamed +5V_AUX
- net +5V_AUX: now also J29.2 (Pin_2)
- removed net USBC_REF: H3.2
- removed net USBC_S: C64.2, H3.1
- net VBUS_C renamed +12V_AUX
- net +12V_AUX: now also F8.2, J28.2 (Pin_2)
- new net +12V_IN_H2: F2.1, J2.2 (Pin_2)
- no-connect marks 2 -> 1
Other:
- moved on the sheet: C2, C3, C4, C5, C7, C8, C9, D1, F1, F2, F3, J1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
