File: PCB/kicad/FilMachine_Mainboard.kicad_sch (KiCad schematic)
At the start: 0 parts

Commit message: new board
Other:
- note added: "Collegamenti per etichette globali: ogni pin ha il nome della sua net. Sorgente: design.py (rigenerare schema e PCB da li'). Display JC4880P433 collegato con flat 2x13 su J5 (pin 1 = pin 1). Il display si alimenta dal flat JP1 (pin 2/4) tramite F7 + D8; la logica della scheda (3,3 V) viene dal display. J28/J29 = uscite 12 V / 5 V di servizio (PTC). J30 = GPIO liberi A6/A7 dell'MCP23017 (= SPARE O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"
- note removed: "Collegamenti per etichette globali: ogni pin ha il nome della sua net. Sorgente: design.py (rigenerare schema e PCB da li'). Display JC4880P433 collegato con flat 2x13 su J4 (pin 1 = pin 1). Il display si alimenta dal flat JP1 (pin 2/4) tramite F7 + D8; J3 = uscita 5 V di servizio."
Changed lines of the file:
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@@
 	(title_block
 		(title "FilMachine Mainboard v1")
-		(date "2026-10-10")
-		(rev "1.0")
+		(date "2026-10-13")
+		(rev "1.1")
 		(company "FilMachine")
 		(comment 1 "Mainboard per JC4880P433 (ESP32-P4) — generata da design.py")
@@
 		)
 	)
-	(text "Collegamenti per etichette globali: ogni pin ha il nome della sua net.\nSorgente: design.py (rigenerare schema e PCB da li').\nDisplay JC4880P433 collegato con flat 2x13 su J4 (pin 1 = pin 1).\nIl display si alimenta dal flat JP1 (pin 2/4) tramite F7 + D8; J3 = uscita 5 V di servizio."
+	(text "Collegamenti per etichette globali: ogni pin ha il nome della sua net.\nSorgente: design.py (rigenerare schema e PCB da li').\nDisplay JC4880P433 collegato con flat 2x13 su J5 (pin 1 = pin 1).\nIl display si alimenta dal flat JP1 (pin 2/4) tramite F7 + D8; la logica della scheda (3,3 V) viene dal display.\nJ28/J29 = uscite 12 V / 5 V di servizio (PTC). J30 = GPIO liberi A6/A7 dell'MCP23017 (= SPARE OUT 1/2).\nTre ingressi 12 V (riscaldatore 1, riscaldatore 2, principale). Parti LCSC/JLCPCB."
 		(exclude_from_sim no)
 		(at 25 160 0)
