File: PCB/kicad/io.kicad_sch (KiCad schematic)
At the start: 64 parts, among them J10 FLOW, J11 HALL, J12 TEMP 1, J13 TEMP 2, J4 DISPLAY JP1, J5 C6 UART, J6 BATH LEVEL, J7 CHEM 1, J8 CHEM 2, J9 CHEM 3, U3 MCP23017-E/SS, U4 MCP3424-E/SL

Commit message: new board
Parts:
- removed J10: FLOW, Connector_JST:JST_XH_B3B-XH-A_1x03_P2.50mm_Vertical, symbol Connector_Generic:Conn_01x03
- removed J13: TEMP 2, Connector_JST:JST_XH_B3B-XH-A_1x03_P2.50mm_Vertical, symbol Connector_Generic:Conn_01x03
- removed J4: DISPLAY JP1, Connector_IDC:IDC-Header_2x13_P2.54mm_Horizontal, symbol Connector_Generic:Conn_02x13_Odd_Even
- removed J5: C6 UART, Connector_PinHeader_2.54mm:PinHeader_1x05_P2.54mm_Vertical, symbol Connector_Generic:Conn_01x05
- removed J6: BATH LEVEL, Connector_JST:JST_XH_B4B-XH-A_1x04_P2.50mm_Vertical, symbol Connector_Generic:Conn_01x04
- removed U4: MCP3424-E/SL, Package_SO:SOIC-14_3.9x8.7mm_P1.27mm, symbol Analog_ADC:MCP3424x-xSL
- added C26: 1nF, Capacitor_SMD:C_0603_1608Metric, symbol Device:C
- added J10: CHEM 3, Connector_JST:JST_XH_B4B-XH-A_1x04_P2.50mm_Vertical, symbol Connector_Generic:Conn_01x04
- added J14: TEMP 2, Connector_JST:JST_XH_B3B-XH-A_1x03_P2.50mm_Vertical, symbol Connector_Generic:Conn_01x03
- added J5: DISPLAY JP1, Connector_IDC:IDC-Header_2x13_P2.54mm_Horizontal, symbol Connector_Generic:Conn_02x13_Odd_Even
- added J6: C6 UART, Connector_PinHeader_2.54mm:PinHeader_1x05_P2.54mm_Vertical, symbol Connector_Generic:Conn_01x05
- added U4: ADS1115, Package_SO:VSSOP-10_3x3mm_P0.5mm, symbol Analog_ADC:ADS1115IDGS
- C13, C14, C15, C16, C17, C18, C19: LCSC (none) -> C14663; Manufacturer Samsung/Murata (generic) -> Samsung/Yageo (JLCPCB basic)
- C20, C21, C22, C23, C24, C25, C27, C28, C29: LCSC (none) -> C1588; Manufacturer Samsung/Murata (generic) -> Samsung/Yageo (JLCPCB basic)
- C62: value 10uF 16V -> 10uF 25V; LCSC (none) -> C15850; MPN MLCC 10uF 16V -> MLCC 10uF 25V; Manufacturer Samsung/Murata (generic) -> Samsung/Yageo (JLCPCB basic)
- D10, D11, D12, D13, D14, D15, D16, D17, D18, D19, D6, D7: value BAT54WS -> 1N5819WS; LCSC (none) -> C191023; MPN BAT54WS -> 1N5819WS; Manufacturer Nexperia/Diodes -> JLCPCB basic
- D8: value B340A -> SS34; LCSC (none) -> C8678; MPN B340A-13-F -> SS34; Manufacturer Diodes Inc -> JLCPCB basic
- F7: LCSC (none) -> C269134; MPN MF-MSMF110-2 -> SMD1812B110TF/33; Manufacturer Bourns -> Brightking
- J11: value HALL -> FLOW; LCSC (none) -> C2316; MPN B3B-XH-A(LF)(SN) -> XH-3A; Manufacturer JST -> BOOMELE
- J12: value TEMP 1 -> HALL; LCSC (none) -> C2316; MPN B3B-XH-A(LF)(SN) -> XH-3A; Manufacturer JST -> BOOMELE
- J13: renamed from C26; value 1nF -> TEMP 1; footprint Capacitor_SMD:C_0603_1608Metric -> Connector_JST:JST_XH_B3B-XH-A_1x03_P2.50mm_Vertical; symbol Device:C -> Connector_Generic:Conn_01x03; LCSC (none) -> C2316; MPN MLCC 1nF -> XH-3A; Manufacturer Samsung/Murata (generic) -> BOOMELE
- J7: value CHEM 1 -> BATH LEVEL; LCSC (none) -> C37815; MPN B4B-XH-A(LF)(SN) -> XH-4A; Manufacturer JST -> BOOMELE
- J8: value CHEM 2 -> CHEM 1; LCSC (none) -> C37815; MPN B4B-XH-A(LF)(SN) -> XH-4A; Manufacturer JST -> BOOMELE
- J9: value CHEM 3 -> CHEM 2; LCSC (none) -> C37815; MPN B4B-XH-A(LF)(SN) -> XH-4A; Manufacturer JST -> BOOMELE
- R10: LCSC (none) -> C22809; Manufacturer Yageo/UniOhm (generic) -> UNI-ROYAL
- R11: LCSC (none) -> C4184; Manufacturer Yageo/UniOhm (generic) -> UNI-ROYAL
- R12, R13, R14, R20, R21, R22, R23, R24, R25, R26, R27, R28, R29, R8: LCSC (none) -> C25804; Manufacturer Yageo/UniOhm (generic) -> UNI-ROYAL
- R16, R6, R7: LCSC (none) -> C23162; Manufacturer Yageo/UniOhm (generic) -> UNI-ROYAL
- R9: LCSC (none) -> C25803; Manufacturer Yageo/UniOhm (generic) -> UNI-ROYAL
- U3: LCSC (none) -> C558584; MPN MCP23017-E/SS -> MCP23017T-E/SS
Connections:
- net 3V3_DISP is gone; now on net +3V3: R16.2
- net +3V3: now also J13.1 (Pin_1), J14.1 (Pin_1), J5.1 (Pin_1), J5.3 (Pin_3), U4.8 (VDD); no longer J12.1 (Pin_1)
- net +5V_SENS: now also J12.1 (Pin_1), J10.1 (Pin_1)
- net 5V_DISP: now also J5.2 (Pin_2), J5.4 (Pin_4)
- net ADC_12V: now also U4.4 (AIN0)
- net ADC_5V: now also U4.5 (AIN1)
- net ADC_PUMP_IA: now also U4.6 (AIN2)
- net ADC_PUMP_IB: now also U4.7 (AIN3)
- net BATH_MAX_IN: now also J5.12 (Pin_12)
- net BATH_MIN_IN: now also J5.14 (Pin_14)
- net C6_IO9: now also J5.24 (Pin_24), J6.4 (Pin_4)
- net C6_PU: now also J5.26 (Pin_26), J6.5 (Pin_5)
- net C6_RXD: now also J5.20 (Pin_20), J6.2 (Pin_2)
- net C6_TXD: now also J5.22 (Pin_22), J6.3 (Pin_3)
- net CHEM2_MIN: now also C26.1; no longer J13.1
- net FLOW_IN: now also J5.7 (Pin_7)
- net GND: now also J13.3 (Pin_3), C26.2, J10.4 (Pin_4), J14.3 (Pin_3), J5.16 (Pin_16), J5.5 (Pin_5), J5.6 (Pin_6), J6.1 (Pin_1), U4.1 (ADDR), U4.3 (GND); no longer J13.2
- net HALL_IN: now also J5.10 (Pin_10)
- net I2C_SCL: now also J5.25 (Pin_25), U4.10 (SCL)
- net I2C_SDA: now also J5.23 (Pin_23), U4.9 (SDA)
- net MOT_ENA: now also J5.19 (Pin_19)
- net MOT_IN1: now also J5.8 (Pin_8)
- net MOT_IN2: now also J5.17 (Pin_17)
- net ONEWIRE: now also J13.2 (Pin_2), J14.2 (Pin_2), J5.15 (Pin_15); no longer J12.2 (Pin_2)
- net PUMP_ENA: now also J5.9 (Pin_9)
- net PUMP_IN1: now also J5.13 (Pin_13)
- net PUMP_IN2: now also J5.11 (Pin_11)
- net SERVO_PWM: now also J5.21 (Pin_21)
- net SNS_BATH_MAX: now also J7.3 (Pin_3)
- net SNS_BATH_MIN: now also J7.2 (Pin_2)
- net SNS_C1_MAX: now also J8.3 (Pin_3); no longer J7.3 (Pin_3)
- net SNS_C1_MIN: now also J8.2 (Pin_2); no longer J7.2 (Pin_2)
- net SNS_C2_MAX: now also J9.3 (Pin_3); no longer J8.3 (Pin_3)
- net SNS_C2_MIN: now also J9.2 (Pin_2); no longer J8.2 (Pin_2)
- net SNS_C3_MAX: now also J10.3 (Pin_3); no longer J9.3 (Pin_3)
- net SNS_C3_MIN: now also J10.2 (Pin_2); no longer J9.2 (Pin_2)
- net SNS_FLOW: now also J11.2 (Pin_2)
- net SNS_HALL: now also J12.2 (Pin_2); no longer J11.2 (Pin_2)
- no-connect marks 4 -> 6

Commit message: new pcb
Parts:
- removed C24, C25, C26, C27, C28, C29: 1nF, Capacitor_SMD:C_0603_1608Metric, symbol Device:C
- removed D15, D16, D17, D18, D19: 1N5819WS, Diode_SMD:D_SOD-323, symbol Device:D_Schottky
- removed J10: CHEM 3, Connector_JST:JST_XH_B4B-XH-A_1x04_P2.50mm_Vertical, symbol Connector_Generic:Conn_01x04
- removed J7: BATH LEVEL, Connector_JST:JST_XH_B4B-XH-A_1x04_P2.50mm_Vertical, symbol Connector_Generic:Conn_01x04
- removed J8: CHEM 1, Connector_JST:JST_XH_B4B-XH-A_1x04_P2.50mm_Vertical, symbol Connector_Generic:Conn_01x04
- removed J9: CHEM 2, Connector_JST:JST_XH_B4B-XH-A_1x04_P2.50mm_Vertical, symbol Connector_Generic:Conn_01x04
- removed R24, R25, R26, R27, R28, R29: 10k, Resistor_SMD:R_0603_1608Metric, symbol Device:R
- J7: renamed from D14; value 1N5819WS -> BATH LEVEL; footprint Diode_SMD:D_SOD-323 -> Connector_JST:JST_XH_B4B-XH-A_1x04_P2.50mm_Vertical; symbol Device:D_Schottky -> Connector_Generic:Conn_01x04; LCSC C191023 -> C37815; MPN 1N5819WS -> XH-4A; Manufacturer JLCPCB basic -> BOOMELE
Connections:
- net SNS_C1_MIN is gone; now on net +5V_SENS: J7.1 (Pin_1)
- net GND: now also J7.4 (Pin_4)
- net SNS_BATH_MAX: now also J7.3 (Pin_3)
- net SNS_BATH_MIN: now also J7.2 (Pin_2)
- net CHEM1_MAX renamed MCP_B1
- net CHEM1_MIN renamed MCP_B0
- net MCP_B0: no longer J7.2 (A)
- net CHEM2_MAX renamed MCP_B3
- net CHEM2_MIN renamed MCP_B2
- net CHEM3_MAX renamed MCP_B5
- net CHEM3_MIN renamed MCP_B4
