File: PCB/kicad/outputs.kicad_sch (KiCad schematic)
At the start: 71 parts, among them J14 VALVES C1 C2, J15 VALVES C3 WB, J16 VALVES WASTE INLET, J17 VALVES SPARE, J18 HEATER 1, J19 HEATER 2, Q1 AO3400A, Q10 AOD4184A, Q2 AO3400A, Q3 AO3400A, Q4 AO3400A, Q5 AO3400A, Q6 AO3400A, Q7 AO3400A, Q8 AO3400A, Q9 AOD4184A, U5 UCC27524D

Commit message: new board
Parts:
- removed D24, D25, D26, D27: B5819W, Diode_SMD:D_SOD-123, symbol Device:D_Schottky
- removed D33, D34, D35: Yellow, LED_SMD:LED_0603_1608Metric, symbol Device:LED
- removed J14: VALVES C1 C2, TerminalBlock_Phoenix:TerminalBlock_Phoenix_PT-1,5-4-3.5-H_1x04_P3.50mm_Horizontal, symbol Connector_Generic:Conn_01x04
- removed J15: VALVES C3 WB, TerminalBlock_Phoenix:TerminalBlock_Phoenix_PT-1,5-4-3.5-H_1x04_P3.50mm_Horizontal, symbol Connector_Generic:Conn_01x04
- removed J16: VALVES WASTE INLET, TerminalBlock_Phoenix:TerminalBlock_Phoenix_PT-1,5-4-3.5-H_1x04_P3.50mm_Horizontal, symbol Connector_Generic:Conn_01x04
- removed J17: VALVES SPARE, TerminalBlock_Phoenix:TerminalBlock_Phoenix_PT-1,5-4-3.5-H_1x04_P3.50mm_Horizontal, symbol Connector_Generic:Conn_01x04
- removed J18: HEATER 1, TerminalBlock_Phoenix:TerminalBlock_Phoenix_MKDS-3-2-5.08_1x02_P5.08mm_Horizontal, symbol Connector_Generic:Conn_01x02
- removed Q10: AOD4184A, Package_TO_SOT_SMD:TO-252-2, symbol Transistor_FET:IPD50R380CE
- removed R34: 100R, Resistor_SMD:R_0603_1608Metric, symbol Device:R
- removed R54, R55, R56: 4.7k, Resistor_SMD:R_0603_1608Metric, symbol Device:R
- added C40: 1uF 50V, Capacitor_SMD:C_0805_2012Metric, symbol Device:C
- added D31: Yellow, LED_SMD:LED_0805_2012Metric, symbol Device:LED
- added D47, D48: 1N5819WS, Diode_SMD:D_SOD-323, symbol Device:D_Schottky
- added J15: VALVE C1, FM:TB_DB301V-3.5-2P, symbol Connector_Generic:Conn_01x02
- added J16: VALVE C2, FM:TB_DB301V-3.5-2P, symbol Connector_Generic:Conn_01x02
- added J20: VALVE INLET, FM:TB_DB301V-3.5-2P, symbol Connector_Generic:Conn_01x02
- added J21: SPARE OUT 1, FM:TB_DB301V-3.5-2P, symbol Connector_Generic:Conn_01x02
- added J22: SPARE OUT 2, FM:TB_DB301V-3.5-2P, symbol Connector_Generic:Conn_01x02
- added J23: HEATER 1, FM:TB_WJ500V-5.08-2P, symbol Connector_Generic:Conn_01x02
- added J24: HEATER 2, FM:TB_WJ500V-5.08-2P, symbol Connector_Generic:Conn_01x02
- added J30: GPIO SPARE, Connector_PinHeader_2.54mm:PinHeader_1x05_P2.54mm_Vertical, symbol Connector_Generic:Conn_01x05
- added Q1, Q2, Q3, Q4, Q5: AO3400A, Package_TO_SOT_SMD:SOT-23, symbol Transistor_FET:AO3400A
- added R31, R32, R33: 100R, Resistor_SMD:R_0603_1608Metric, symbol Device:R
- added R41, R42, R43, R44: 100k, Resistor_SMD:R_0603_1608Metric, symbol Device:R
- added R97, R98: 1k, Resistor_SMD:R_0603_1608Metric, symbol Device:R
- C41: LCSC (none) -> C14663; Manufacturer Samsung/Murata (generic) -> Samsung/Yageo (JLCPCB basic)
- D21, D22, D23, D28: LCSC (none) -> C8598; MPN B5819W -> B5819W SL; Manufacturer Diodes/CJ -> JLCPCB basic
- D24: renamed from D31; value Yellow -> B5819W; footprint LED_SMD:LED_0603_1608Metric -> Diode_SMD:D_SOD-123; symbol Device:LED -> Device:D_Schottky; LCSC (none) -> C8598; MPN KT-0603Y -> B5819W SL; Manufacturer Hubei KENTO -> JLCPCB basic
- D25: renamed from R33; value 100R -> B5819W; footprint Resistor_SMD:R_0603_1608Metric -> Diode_SMD:D_SOD-123; symbol Device:R -> Device:D_Schottky; LCSC (none) -> C8598; MPN 0603 100R 1% -> B5819W SL; Manufacturer Yageo/UniOhm (generic) -> JLCPCB basic
- D26: renamed from R44; value 100k -> B5819W; footprint Resistor_SMD:R_0603_1608Metric -> Diode_SMD:D_SOD-123; symbol Device:R -> Device:D_Schottky; LCSC (none) -> C8598; MPN 0603 100k 1% -> B5819W SL; Manufacturer Yageo/UniOhm (generic) -> JLCPCB basic
- D27: renamed from Q5; value AO3400A -> B5819W; footprint Package_TO_SOT_SMD:SOT-23 -> Diode_SMD:D_SOD-123; symbol Transistor_FET:AO3400A -> Device:D_Schottky; LCSC (none) -> C8598; MPN AO3400A -> B5819W SL; Manufacturer Alpha & Omega -> JLCPCB basic
- D32, D36, D37, D38: footprint LED_SMD:LED_0603_1608Metric -> LED_SMD:LED_0805_2012Metric; LCSC (none) -> C2296; MPN KT-0603Y -> KT-0805Y
- D33: renamed from R31; value 100R -> Yellow; footprint Resistor_SMD:R_0603_1608Metric -> LED_SMD:LED_0805_2012Metric; symbol Device:R -> Device:LED; LCSC (none) -> C2296; MPN 0603 100R 1% -> KT-0805Y; Manufacturer Yageo/UniOhm (generic) -> Hubei KENTO
- D34: renamed from R42; value 100k -> Yellow; footprint Resistor_SMD:R_0603_1608Metric -> LED_SMD:LED_0805_2012Metric; symbol Device:R -> Device:LED; LCSC (none) -> C2296; MPN 0603 100k 1% -> KT-0805Y; Manufacturer Yageo/UniOhm (generic) -> Hubei KENTO
- D35: renamed from Q3; value AO3400A -> Yellow; footprint Package_TO_SOT_SMD:SOT-23 -> LED_SMD:LED_0805_2012Metric; symbol Transistor_FET:AO3400A -> Device:LED; LCSC (none) -> C2296; MPN AO3400A -> KT-0805Y; Manufacturer Alpha & Omega -> Hubei KENTO
- D41, D42: LCSC (none) -> C8678; Manufacturer MDD/onsemi -> JLCPCB basic
- D43, D44: LCSC (none) -> C2286
- J17: renamed from R41; value 100k -> VALVE C3; footprint Resistor_SMD:R_0603_1608Metric -> FM:TB_DB301V-3.5-2P; symbol Device:R -> Connector_Generic:Conn_01x02; LCSC (none) -> C695629; MPN 0603 100k 1% -> DB301V-3.5-2P-GN-S; Manufacturer Yageo/UniOhm (generic) -> DORABO
- J18: renamed from Q2; value AO3400A -> VALVE WB; footprint Package_TO_SOT_SMD:SOT-23 -> FM:TB_DB301V-3.5-2P; symbol Transistor_FET:AO3400A -> Connector_Generic:Conn_01x02; LCSC (none) -> C695629; MPN AO3400A -> DB301V-3.5-2P-GN-S; Manufacturer Alpha & Omega -> DORABO
- J19: value HEATER 2 -> VALVE WASTE; footprint TerminalBlock_Phoenix:TerminalBlock_Phoenix_MKDS-3-2-5.08_1x02_P5.08mm_Horizontal -> FM:TB_DB301V-3.5-2P; LCSC (none) -> C695629; MPN 1711026 -> DB301V-3.5-2P-GN-S; Manufacturer Phoenix Contact -> DORABO
- Q10: renamed from C40; value 1uF 25V -> AOD4184A; footprint Capacitor_SMD:C_0805_2012Metric -> Package_TO_SOT_SMD:TO-252-2; symbol Device:C -> Transistor_FET:IPD50R380CE; LCSC (none) -> C99124; MPN MLCC 1uF 25V -> AOD4184A; Manufacturer Samsung/Murata (generic) -> Alpha & Omega
- Q6, Q7, Q8: LCSC (none) -> C20917
- Q9: LCSC (none) -> C99124
- R34: renamed from Q1; value AO3400A -> 100R; footprint Package_TO_SOT_SMD:SOT-23 -> Resistor_SMD:R_0603_1608Metric; symbol Transistor_FET:AO3400A -> Device:R; LCSC (none) -> C22775; MPN AO3400A -> 0603 100R 1%; Manufacturer Alpha & Omega -> UNI-ROYAL
- R35, R36, R37, R38: LCSC (none) -> C22775; Manufacturer Yageo/UniOhm (generic) -> UNI-ROYAL
- R45, R46, R61, R62: LCSC (none) -> C25803; Manufacturer Yageo/UniOhm (generic) -> UNI-ROYAL
- R47, R48: value 100k -> 1M; LCSC (none) -> C22935; MPN 0603 100k 1% -> 0603 1M 1%; Manufacturer Yageo/UniOhm (generic) -> UNI-ROYAL
- R51, R52, R53, R57, R58, R67, R68: LCSC (none) -> C23162; Manufacturer Yageo/UniOhm (generic) -> UNI-ROYAL
- R54: renamed from R32; value 100R -> 4.7k; LCSC (none) -> C23162; MPN 0603 100R 1% -> 0603 4.7k 1%; Manufacturer Yageo/UniOhm (generic) -> UNI-ROYAL
- R55: renamed from R43; value 100k -> 4.7k; LCSC (none) -> C23162; MPN 0603 100k 1% -> 0603 4.7k 1%; Manufacturer Yageo/UniOhm (generic) -> UNI-ROYAL
- R56: renamed from Q4; value AO3400A -> 4.7k; footprint Package_TO_SOT_SMD:SOT-23 -> Resistor_SMD:R_0603_1608Metric; symbol Transistor_FET:AO3400A -> Device:R; LCSC (none) -> C23162; MPN AO3400A -> 0603 4.7k 1%; Manufacturer Alpha & Omega -> UNI-ROYAL
- R63, R65: LCSC (none) -> C22859; Manufacturer Yageo/UniOhm (generic) -> UNI-ROYAL
- R64, R66: LCSC (none) -> C25804; Manufacturer Yageo/UniOhm (generic) -> UNI-ROYAL
- U5: LCSC (none) -> C465729
Connections:
- net +12V: now also D24.1 (K), D25.1 (K), D26.1 (K), D27.1 (K), J17.1 (Pin_1), J18.1 (Pin_1), J19.1 (Pin_1), R54.1, R55.1, R56.1, C40.1, J15.1 (Pin_1), J16.1 (Pin_1), J20.1 (Pin_1), J21.1 (Pin_1), J22.1 (Pin_1); no longer Q10.1
- net +12V_H1: now also J23.2 (Pin_2)
- net +12V_H2: now also J24.2 (Pin_2); no longer J19.2 (Pin_2)
- net GND: now also Q10.3 (S), C40.2, J30.5 (Pin_5), Q1.2 (S), Q2.2 (S), Q3.2 (S), Q4.2 (S), Q5.2 (S), R41.2, R42.2, R43.2, R44.2; no longer D26.2, D27.2 (S), D34.2, D35.2 (S), J17.2, J18.2 (S), Q10.2, R34.2 (S), R55.2, R56.2 (S)
- net HEAT1_N: now also J23.1 (Pin_1)
- net HEAT2_G: now also Q10.1 (G)
- net HEAT2_N: now also Q10.2 (D), J24.1 (Pin_1); no longer J19.1 (Pin_1)
- net VLV1_G: now also Q1.1 (G), R31.2, R41.1; no longer D33.2, J17.1, R34.1 (G)
- net VLV1_LED: now also D31.2 (A); no longer D24.2 (A)
- net VLV1_N: now also D31.1 (K), J15.2 (Pin_2), Q1.3 (D); no longer D24.1 (K), R34.3 (D)
- net VLV2_G: now also Q2.1 (G), R32.2, R42.1; no longer D34.1, J18.1 (G), R54.2
- net VLV2_N: now also J16.2 (Pin_2), Q2.3 (D); no longer J18.3 (D)
- net VLV3_G: now also Q3.1 (G), R33.2, R43.1; no longer D25.2, D35.1 (G), R55.1
- net VLV3_LED: now also D33.2 (A)
- net VLV3_N: now also D33.1 (K), J17.2 (Pin_2), Q3.3 (D); no longer D35.3 (D)
- net VLV4_G: now also R34.2, Q4.1 (G), R44.1; no longer D26.1, R56.1 (G)
- net VLV4_LED: now also D34.2 (A), R54.2
- net VLV4_N: now also D24.2 (A), D34.1 (K), J18.2 (Pin_2), Q4.3 (D); no longer R56.3 (D)
- net VLV5_G: now also Q5.1 (G); no longer D27.1 (G)
- net VLV5_LED: now also D35.2 (A), R55.2
- net VLV5_N: now also D25.2 (A), D35.1 (K), J19.2 (Pin_2), Q5.3 (D); no longer D27.3 (D)
- net VLV6_LED: now also R56.2
- net VLV6_N: now also D26.2 (A), J20.2 (Pin_2)
- net VLV7_N: now also D27.2 (A), J21.2 (Pin_2)
- net VLV8_N: now also J22.2 (Pin_2)
- net VLV_C1: now also R31.1; no longer D33.1
- net VLV_C2: now also R32.1; no longer R54.1
- net VLV_C3: now also R33.1; no longer D25.1
- net VLV_SP1: now also R97.1
- net VLV_SP2: now also R98.1
- net VLV_WB: now also R34.1
- new net +3V3: D47.1 (K), D48.1 (K), J30.3 (Pin_3)
- new net +5V_AUX: J30.4 (Pin_4)
- new net SP1_IO: D47.2 (A), J30.1 (Pin_1), R97.2
- new net SP2_IO: D48.2 (A), J30.2 (Pin_2), R98.2
Other:
- moved on the sheet: R54, R55

Commit message: new pcb
Parts:
- removed D42: SS34, Diode_SMD:D_SMA, symbol Device:D_Schottky
- removed D44: Red, LED_SMD:LED_0603_1608Metric, symbol Device:LED
- removed J24: HEATER 2, FM:TB_WJ500V-5.08-2P, symbol Connector_Generic:Conn_01x02
- removed J30: GPIO SPARE, Connector_PinHeader_2.54mm:PinHeader_1x05_P2.54mm_Vertical, symbol Connector_Generic:Conn_01x05
- removed R68: 4.7k, Resistor_SMD:R_0603_1608Metric, symbol Device:R
- added C41: 100nF, Capacitor_SMD:C_0603_1608Metric, symbol Device:C
- added D49, D50, D51, D52: 1N5819WS, Diode_SMD:D_SOD-323, symbol Device:D_Schottky
- added J30: GPIO SPARE, Connector_PinHeader_2.54mm:PinHeader_1x09_P2.54mm_Vertical, symbol Connector_Generic:Conn_01x09
- added R100, R101, R102, R99: 1k, Resistor_SMD:R_0603_1608Metric, symbol Device:R
- added R61, R62: 100k, Resistor_SMD:R_0603_1608Metric, symbol Device:R
- added R63: 10R, Resistor_SMD:R_0603_1608Metric, symbol Device:R
- D42: renamed from C41; value 100nF -> SS34; footprint Capacitor_SMD:C_0603_1608Metric -> Diode_SMD:D_SMA; symbol Device:C -> Device:D_Schottky; LCSC C14663 -> C8678; MPN MLCC 100nF -> SS34; Manufacturer Samsung/Yageo (JLCPCB basic) -> JLCPCB basic
- D44: renamed from R62; value 100k -> Red; footprint Resistor_SMD:R_0603_1608Metric -> LED_SMD:LED_0603_1608Metric; symbol Device:R -> Device:LED; LCSC C25803 -> C2286; MPN 0603 100k 1% -> KT-0603R; Manufacturer UNI-ROYAL -> Hubei KENTO
- J24: renamed from R63; value 10R -> HEATER 2; footprint Resistor_SMD:R_0603_1608Metric -> FM:TB_WJ500V-5.08-2P; symbol Device:R -> Connector_Generic:Conn_01x02; LCSC C22859 -> C8465; MPN 0603 10R 1% -> WJ500V-5.08-2P; Manufacturer UNI-ROYAL -> Ningbo Kangnex
- R47, R48: value 1M -> 100k; LCSC C22935 -> C25803; MPN 0603 1M 1% -> 0603 100k 1%
- R68: renamed from R61; value 100k -> 4.7k; LCSC C25803 -> C23162; MPN 0603 100k 1% -> 0603 4.7k 1%
Connections:
- net +12V: now also C41.1; no longer D42.1
- net +12V_H2: now also D42.1 (K), J24.2 (Pin_2)
- net +3V3: now also D49.1 (K), D50.1 (K), D51.1 (K), D52.1 (K), J30.7 (Pin_7)
- net +5V_AUX: now also J30.8 (Pin_8)
- net GND: now also D44.1 (K), C41.2, J30.9 (Pin_9), R61.2, R62.2; no longer D42.2, D44.2, R68.2
- net HEAT1_CMD: now also R61.1; no longer R68.1
- net HEAT1_DRV: now also R63.1; no longer J24.1
- net HEAT1_G: now also R63.2; no longer J24.2
- net HEAT2_CMD: now also R62.1; no longer D44.1
- net HEAT2_DRV: now also R68.1
- net HEAT2_LED: now also D44.2 (A), R68.2
- net HEAT2_N: now also D42.2 (A), J24.1 (Pin_1)
- net VLV_SP1: no longer R97.1
- net VLV_SP2: no longer R98.1
- net SP1_IO renamed SPB0_IO
- net SPB0_IO: now also J30.1 (Pin_1)
- net SP2_IO renamed SPB1_IO
- net SPB1_IO: now also J30.2 (Pin_2)
- new net MCP_B0: R97.1
- new net MCP_B1: R98.1
- new net MCP_B2: R99.1
- new net MCP_B3: R100.1
- new net MCP_B4: R101.1
- new net MCP_B5: R102.1
- new net SPB2_IO: D49.2 (A), J30.3 (Pin_3), R99.2
- new net SPB3_IO: D50.2 (A), J30.4 (Pin_4), R100.2
- new net SPB4_IO: D51.2 (A), J30.5 (Pin_5), R101.2
- new net SPB5_IO: D52.2 (A), J30.6 (Pin_6), R102.2
Other:
- moved on the sheet: R68
