File: PCB/kicad/FilMachine_Mainboard.kicad_pcb (KiCad board)
At the start: 4 copper layers, 110 x 90 mm, 223 parts, among them J1 12V HEAT IN, J10 FLOW, J11 HALL, J12 TEMP 1, J13 TEMP 2, J14 VALVES C1 C2, J15 VALVES C3 WB, J16 VALVES WASTE INLET, J17 VALVES SPARE, J18 HEATER 1, J19 HEATER 2, J2 12V MAIN IN, J20 PUMP, J21 MOTOR, J22 SERVO, J3 USB-C 5V OUT, J4 DISPLAY JP1, J5 C6 UART, J6 BATH LEVEL, J7 CHEM 1, J8 CHEM 2, J9 CHEM 3, Q1 AO3400A, Q10 AOD4184A, Q11 AO3401A, Q12 AO3401A, Q2 AO3400A, Q3 AO3400A, Q4 AO3400A, Q5 AO3400A, Q6 AO3400A, Q7 AO3400A, Q8 AO3400A, Q9 AOD4184A, U1 LMR33630ADDA, U10 DRV8871DDA, U11 TLV7041, U2 AP2112K-3.3, U3 MCP23017-E/SS, U4 MCP3424-E/SL, U5 UCC27524D, U6 74LVC2G08, U7 74LVC2G08, U8 BTN8982TA, U9 BTN8982TA

Commit message: new board
Parts:
- removed C11: 1uF 16V, Capacitor_SMD:C_0603_1608Metric
- removed C12: 2.2uF 16V, Capacitor_SMD:C_0603_1608Metric
- removed C65: 100nF, Capacitor_SMD:C_0603_1608Metric
- removed D45, D46: 1N4148WS, Diode_SMD:D_SOD-323
- removed J4: DISPLAY JP1, Connector_IDC:IDC-Header_2x13_P2.54mm_Horizontal
- removed Q11, Q12: AO3401A, Package_TO_SOT_SMD:SOT-23
- removed R89, R90: 56k, Resistor_SMD:R_0603_1608Metric
- removed R91: 220k, Resistor_SMD:R_0603_1608Metric
- removed R92, R96: 10k, Resistor_SMD:R_0603_1608Metric
- removed R93: 130k, Resistor_SMD:R_0603_1608Metric
- removed R94, R95: 100k, Resistor_SMD:R_0603_1608Metric
- removed U11: TLV7041, Package_TO_SOT_SMD:SOT-23-5
- removed U2: AP2112K-3.3, Package_TO_SOT_SMD:SOT-23-5
- added D47: 1N5819WS, Diode_SMD:D_SOD-323, F.Cu at (158.1, 137.1)
- added D48: 1N5819WS, Diode_SMD:D_SOD-323, F.Cu at (158.1, 139.3)
- added F8: 2A, Fuse:Fuse_1812_4532Metric, F.Cu at (187.0, 109.8)
- added J23: HEATER 1, FM:TB_WJ500V-5.08-2P, F.Cu at (118.6, 105.3)
- added J24: HEATER 2, FM:TB_WJ500V-5.08-2P, F.Cu at (132.6, 105.3)
- added J25: PUMP, FM:TB_WJ500V-5.08-2P, F.Cu at (105.3, 159.4)
- added J26: MOTOR, FM:TB_DB301V-3.5-2P, F.Cu at (112.8, 186.3)
- added J27: SERVO, Connector_PinHeader_2.54mm:PinHeader_1x03_P2.54mm_Vertical, F.Cu at (178.8, 154.4)
- added J28: 12V OUT, FM:TB_DB301V-3.5-2P, F.Cu at (188.0, 103.7)
- added J29: 5V OUT, FM:TB_DB301V-3.5-2P, F.Cu at (195.8, 103.7)
- added J30: GPIO SPARE, Connector_PinHeader_2.54mm:PinHeader_1x05_P2.54mm_Vertical, F.Cu at (155.0, 142.3)
- added R97: 1k, Resistor_SMD:R_0603_1608Metric, F.Cu at (154.7, 136.9)
- added R98: 1k, Resistor_SMD:R_0603_1608Metric, F.Cu at (154.7, 139.1)
- C1: value 100uF 25V -> 100uF 35V; footprint Capacitor_THT:CP_Radial_D8.0mm_P3.50mm -> Capacitor_THT:CP_Radial_D6.3mm_P2.50mm
- C10, C7, C8, C9: value 22uF 16V -> 22uF 25V
- C2, C3, C57, C59: footprint Capacitor_SMD:C_1210_3225Metric -> Capacitor_SMD:C_1206_3216Metric
- C4: footprint Capacitor_SMD:C_0603_1608Metric -> Capacitor_SMD:C_0805_2012Metric
- C40: value 1uF 25V -> 1uF 50V
- C6: value 1uF 16V -> 1uF 50V
- C60: value 100uF 10V -> 47uF 10V; footprint Capacitor_SMD:C_1210_3225Metric -> Capacitor_SMD:C_1206_3216Metric
- C62: value 10uF 16V -> 10uF 25V
- C63: value 4.7uF 16V -> 10uF 25V
- C64: value 100nF -> 10uF 25V; footprint Capacitor_SMD:C_0603_1608Metric -> Capacitor_SMD:C_0805_2012Metric
- D1, D2: value SMCJ16A -> SMBJ16A; footprint Diode_SMD:D_SMC -> Diode_SMD:D_SMB
- D10, D11, D12, D13, D14, D15, D16, D17, D18, D19, D6, D7: value BAT54WS -> 1N5819WS
- D3, D31, D32, D33, D34, D35, D36, D37, D38, D4, D5: footprint LED_SMD:LED_0603_1608Metric -> LED_SMD:LED_0805_2012Metric
- D8: value B340A -> SS34
- F1, F2, F3: value 15A MINI -> 15A; footprint Fuse:Fuseholder_Blade_Mini_Keystone_3568 -> FM:FUSE_2410_SMD
- F4: value 7.5A MINI -> 8A; footprint Fuse:Fuseholder_Blade_Mini_Keystone_3568 -> FM:FUSE_2410_SMD
- F5: value 1.5A -> 1.1A
- J1: value 12V HEAT IN -> 12V IN HEATER 1; footprint TerminalBlock_Phoenix:TerminalBlock_Phoenix_MKDS-3-2-5.08_1x02_P5.08mm_Horizontal -> FM:TB_WJ500V-5.08-2P
- J10: value FLOW -> CHEM 3; footprint Connector_JST:JST_XH_B3B-XH-A_1x03_P2.50mm_Vertical -> Connector_JST:JST_XH_B4B-XH-A_1x04_P2.50mm_Vertical
- J11: value HALL -> FLOW
- J12: value TEMP 1 -> HALL
- J13: value TEMP 2 -> TEMP 1
- J14: value VALVES C1 C2 -> TEMP 2; footprint TerminalBlock_Phoenix:TerminalBlock_Phoenix_PT-1,5-4-3.5-H_1x04_P3.50mm_Horizontal -> Connector_JST:JST_XH_B3B-XH-A_1x03_P2.50mm_Vertical
- J15: value VALVES C3 WB -> VALVE C1; footprint TerminalBlock_Phoenix:TerminalBlock_Phoenix_PT-1,5-4-3.5-H_1x04_P3.50mm_Horizontal -> FM:TB_DB301V-3.5-2P
- J16: value VALVES WASTE INLET -> VALVE C2; footprint TerminalBlock_Phoenix:TerminalBlock_Phoenix_PT-1,5-4-3.5-H_1x04_P3.50mm_Horizontal -> FM:TB_DB301V-3.5-2P
- J17: value VALVES SPARE -> VALVE C3; footprint TerminalBlock_Phoenix:TerminalBlock_Phoenix_PT-1,5-4-3.5-H_1x04_P3.50mm_Horizontal -> FM:TB_DB301V-3.5-2P
- J18: value HEATER 1 -> VALVE WB; footprint TerminalBlock_Phoenix:TerminalBlock_Phoenix_MKDS-3-2-5.08_1x02_P5.08mm_Horizontal -> FM:TB_DB301V-3.5-2P
- J19: value HEATER 2 -> VALVE WASTE; footprint TerminalBlock_Phoenix:TerminalBlock_Phoenix_MKDS-3-2-5.08_1x02_P5.08mm_Horizontal -> FM:TB_DB301V-3.5-2P
- J2: value 12V MAIN IN -> 12V IN HEATER 2; footprint TerminalBlock_Phoenix:TerminalBlock_Phoenix_MKDS-3-2-5.08_1x02_P5.08mm_Horizontal -> FM:TB_WJ500V-5.08-2P
- J20: value PUMP -> VALVE INLET; footprint TerminalBlock_Phoenix:TerminalBlock_Phoenix_MKDS-3-2-5.08_1x02_P5.08mm_Horizontal -> FM:TB_DB301V-3.5-2P
- J21: value MOTOR -> SPARE OUT 1; footprint TerminalBlock_Phoenix:TerminalBlock_Phoenix_PT-1,5-2-3.5-H_1x02_P3.50mm_Horizontal -> FM:TB_DB301V-3.5-2P
- J22: value SERVO -> SPARE OUT 2; footprint Connector_PinHeader_2.54mm:PinHeader_1x03_P2.54mm_Vertical -> FM:TB_DB301V-3.5-2P
- J3: value USB-C 5V OUT -> 12V IN MAIN; footprint Connector_USB:USB_C_Receptacle_GCT_USB4125-xx-x_6P_TopMnt_Horizontal -> FM:TB_WJ500V-5.08-2P
- J5: value C6 UART -> DISPLAY JP1; footprint Connector_PinHeader_2.54mm:PinHeader_1x05_P2.54mm_Vertical -> Connector_IDC:IDC-Header_2x13_P2.54mm_Horizontal
- J6: value BATH LEVEL -> C6 UART; footprint Connector_JST:JST_XH_B4B-XH-A_1x04_P2.50mm_Vertical -> Connector_PinHeader_2.54mm:PinHeader_1x05_P2.54mm_Vertical
- J7: value CHEM 1 -> BATH LEVEL
- J8: value CHEM 2 -> CHEM 1
- J9: value CHEM 3 -> CHEM 2
- L1: value 6.8uH -> 10uH; footprint Inductor_SMD:L_Bourns_SRP7028A_7.3x6.6mm -> FM:L_SLO0630H
- R2: value 24.3k -> 24k
- R47, R48: value 100k -> 1M
- R84: value 10k -> 1k
- U4: value MCP3424-E/SL -> ADS1115; footprint Package_SO:SOIC-14_3.9x8.7mm_P1.27mm -> Package_SO:VSSOP-10_3x3mm_P0.5mm
- U8, U9: value BTN8982TA -> BTN8962TA
- moved J3 94.7 mm to (105.3, 141.4), turned to -90 degrees
- moved J18 92.9 mm to (167.6, 186.3), turned to 0 degrees
- moved J19 89.8 mm to (175.2, 186.3), turned to 0 degrees
- moved J20 82.3 mm to (182.8, 186.3), turned to 0 degrees
- moved J21 79.1 mm to (190.4, 186.3)
- moved J14 62.5 mm to (198.5, 155.0), turned to 90 degrees
- moved F5 56.6 mm to (197.0, 109.8)
- moved J6 54.7 mm to (163.8, 154.4)
- moved J5 43.7 mm to (147.6, 113.8)
- moved J11 42.6 mm to (205.9, 173.0)
- moved J22 37.2 mm to (198.0, 186.3), turned to 0 degrees
- moved J17 29.5 mm to (160.0, 186.3)
- moved J2 25.7 mm to (105.3, 113.4)
- moved J16 21.8 mm to (152.4, 186.3)
- moved J15 14.1 mm to (144.8, 186.3)
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Connections:
- C63 pad 1: VBUS_C -> +12V_AUX
- C64 pad 1: USBC_GATE -> +5V_AUX
- C64 pad 2: USBC_S -> GND
- F1 pad 1: +12V_IN_H -> +12V_IN_H1
- F2 pad 1: +12V_IN_H -> +12V_IN_H2
- F5 pad 2: +5V_USB -> +5V_AUX
- J1 pad 2: +12V_IN_H -> +12V_IN_H1
- J10 pad 2: SNS_FLOW -> SNS_C3_MIN
- J10 pad 3: GND -> SNS_C3_MAX
- J11 pad 2: SNS_HALL -> SNS_FLOW
- J12 pad 1: +3V3 -> +5V_SENS
- J12 pad 2: ONEWIRE -> SNS_HALL
- J14 pad 1: +12V -> +3V3
- J14 pad 2: VLV1_N -> ONEWIRE
- J14 pad 3: +12V -> GND
- J15 pad 2: VLV3_N -> VLV1_N
- J16 pad 2: VLV5_N -> VLV2_N
- J17 pad 2: VLV7_N -> VLV3_N
- J18 pad 1: HEAT1_N -> +12V
- J18 pad 2: +12V_H1 -> VLV4_N
- J19 pad 1: HEAT2_N -> +12V
- J19 pad 2: +12V_H2 -> VLV5_N
- J2 pad 2: +12V_IN_M -> +12V_IN_H2
- J20 pad 1: PUMP_OUT_A -> +12V
- J20 pad 2: PUMP_OUT_B -> VLV6_N
- J21 pad 1: MOT_OUT_A -> +12V
- J21 pad 2: MOT_OUT_B -> VLV7_N
- J22 pad 1: SERVO_SIG -> +12V
- J22 pad 2: +5V -> VLV8_N
- J5 pad 1: GND -> +3V3
- J5 pad 2: C6_RXD -> 5V_DISP
- J5 pad 3: C6_TXD -> +3V3
- J5 pad 4: C6_IO9 -> 5V_DISP
- J5 pad 5: C6_PU -> GND
- J6 pad 1: +5V_SENS -> GND
- J6 pad 2: SNS_BATH_MIN -> C6_RXD
- J6 pad 3: SNS_BATH_MAX -> C6_TXD
- J6 pad 4: GND -> C6_IO9
- J7 pad 2: SNS_C1_MIN -> SNS_BATH_MIN
- J7 pad 3: SNS_C1_MAX -> SNS_BATH_MAX
- J8 pad 2: SNS_C2_MIN -> SNS_C1_MIN
- J8 pad 3: SNS_C2_MAX -> SNS_C1_MAX
- J9 pad 2: SNS_C3_MIN -> SNS_C2_MIN
- J9 pad 3: SNS_C3_MAX -> SNS_C2_MAX
- R16 pad 2: 3V3_DISP -> +3V3
- U4 pad 1: ADC_12V -> GND
- U4 pad 10: GND -> I2C_SCL
- U4 pad 2: GND -> (no net)
- U4 pad 3: ADC_5V -> GND
- U4 pad 4: GND -> ADC_12V
- U4 pad 5: GND -> ADC_5V
- U4 pad 6: +3V3 -> ADC_PUMP_IA
- U4 pad 7: I2C_SDA -> ADC_PUMP_IB
- U4 pad 8: I2C_SCL -> +3V3
- U4 pad 9: GND -> I2C_SDA
Routing:
- net +5V_AUX: track 0.00 -> 89.5 mm, vias 0 -> 2
- net SNS_C1_MIN: track 115.2 -> 36.3 mm, vias 6 -> 2
- net CHEM3_MIN: track 18.9 -> 96.4 mm, vias 0 -> 3
- net +5V_USB: track 70.7 -> 0.00 mm, vias 6 -> 0
- net 3V3_DISP: track 63.4 -> 0.00 mm, vias 1 -> 0
- net C6_TXD: track 45.5 -> 100.3 mm, vias 0 -> 4
- net VLV_SP2: track 68.2 -> 117.2 mm, vias 4 -> 9
- net CHEM2_MAX: track 44.9 -> 91.5 mm, vias 3 -> 9
- net +5V: track 118.3 -> 160.6 mm
- net HEAT1_DRV: track 16.8 -> 53.0 mm, vias 0 -> 4
- net CHEM2_MIN: track 73.8 -> 38.7 mm, vias 8 -> 4
- net HALL_IN: track 72.7 -> 38.8 mm, vias 2 -> 3
- net USBC_S: track 32.3 -> 0.00 mm
- net VLV_C1: track 42.7 -> 74.9 mm
- net VLV_SP1: track 70.8 -> 102.8 mm, vias 6 -> 8
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- added copper zone on F.Cu, net +12V_IN_H1
- added copper zone on B.Cu, net +12V_IN_H2
- added copper zone on F.Cu, net +12V_IN_H2
- added copper zone on In2.Cu, net +12V_IN_H2
- removed copper zone on B.Cu, net +12V_H1
- removed copper zone on B.Cu, net +12V_H2
- removed copper zone on B.Cu, net +12V_IN_H
- removed copper zone on F.Cu, net +12V_IN_H
- removed copper zone on In2.Cu, net +12V_IN_H
- removed copper zone on B.Cu, net +12V_IN_M
- removed copper zone on In2.Cu, net +12V_IN_M
- removed copper zone on B.Cu, net HEAT1_N
- removed copper zone on B.Cu, net HEAT2_N
- removed copper zone on B.Cu, net PUMP_OUT_A
- removed copper zone on B.Cu, net PUMP_OUT_B
Other:
- board text added: "+"
- board text added: "+ 12V IN HEATER 1 -"
- board text added: "+ 12V IN HEATER 2 -"
- board text added: "+ 12V IN MAIN -"
- board text added: "+ a sinistra, - a destra"
- board text added: "-"
- board text added: "15A"
- board text added: "3V3"
- board text added: "5V"
- board text added: "8A"
- board text added: "A6"
- board text added: "A7"
- board text added: "B PUMP A"
- board text added: "Board v1.1"
- board text added: "C1"
- board text added: "C2"
- board text added: "C3"
- board text added: "FilMachine Board v1.1 - 2026-10"
- board text added: "GND"
- board text added: "GPIO SPARE"
- board text added: "INLET"
- board text added: "JLCJLCJLCJLC"
- board text added: "SPARE 1"
- board text added: "SPARE 2"
- board text added: "VALVOLE 12V: + sx - dx"
- board text added: "WASTE"
- board text added: "WB"
- board text added: "sx 12V OUT 2A dx 5V OUT 1A"
- board text removed: "+ sotto"
- board text removed: "- sopra"
- board text removed: "- sopra + sotto"
- board text removed: "12V HEAT IN"
- board text removed: "12V MAIN IN"
- board text removed: "5V OUT"
- board text removed: "Board v1.0"
- board text removed: "FilMachine Board v1.0 - 2026-10"
- board text removed: "PUMP"
- board text removed: "SPARE A6 | A7"
- board text removed: "USB-C"
- board text removed: "VALVE C1 | C2"
- board text removed: "VALVE C3 | WB"
- board text removed: "WASTE | INLET"

Commit message: new pcb
Parts:
- removed C24, C25, C26, C27, C28, C29: 1nF, Capacitor_SMD:C_0603_1608Metric
- removed D14, D15, D16, D17, D18, D19: 1N5819WS, Diode_SMD:D_SOD-323
- removed J10: CHEM 3, Connector_JST:JST_XH_B4B-XH-A_1x04_P2.50mm_Vertical
- removed J8: CHEM 1, Connector_JST:JST_XH_B4B-XH-A_1x04_P2.50mm_Vertical
- removed J9: CHEM 2, Connector_JST:JST_XH_B4B-XH-A_1x04_P2.50mm_Vertical
- removed R24, R25, R26, R27, R28, R29: 10k, Resistor_SMD:R_0603_1608Metric
- added D49: 1N5819WS, Diode_SMD:D_SOD-323, F.Cu at (193.8, 126.4)
- added D50: 1N5819WS, Diode_SMD:D_SOD-323, F.Cu at (176.8, 128.6)
- added D51: 1N5819WS, Diode_SMD:D_SOD-323, F.Cu at (183.7, 128.6)
- added D52: 1N5819WS, Diode_SMD:D_SOD-323, F.Cu at (190.5, 128.6)
- added R100: 1k, Resistor_SMD:R_0603_1608Metric, F.Cu at (197.2, 126.2)
- added R101: 1k, Resistor_SMD:R_0603_1608Metric, F.Cu at (180.3, 128.4)
- added R102: 1k, Resistor_SMD:R_0603_1608Metric, F.Cu at (187.1, 128.4)
- added R99: 1k, Resistor_SMD:R_0603_1608Metric, F.Cu at (190.4, 126.2)
- J30: footprint Connector_PinHeader_2.54mm:PinHeader_1x05_P2.54mm_Vertical -> Connector_PinHeader_2.54mm:PinHeader_1x09_P2.54mm_Vertical
- R47, R48: value 1M -> 100k
- moved J11 39.5 mm to (205.9, 133.5)
- moved D48 31.6 mm to (187.0, 126.4)
- moved R98 31.6 mm to (183.6, 126.2)
- moved J30 24.5 mm to (177.8, 133.4), turned to 90 degrees
- moved D47 24.5 mm to (180.1, 126.4)
- moved R97 24.5 mm to (176.7, 126.2)
- moved J14 21.8 mm to (205.9, 175.5)
- moved J13 19.9 mm to (205.9, 161.5)
- moved J12 18.1 mm to (205.9, 147.5)
- moved R16 6.72 mm to (176.7, 123.3)
- moved C64 1.60 mm to (185.7, 114.7)
- moved C63 1.60 mm to (192.0, 110.4)
- moved F5 1.60 mm to (197.0, 111.4)
- moved F8 1.60 mm to (187.0, 111.4)
- turned R62 to 180 degrees
Connections:
- net SP1_IO renamed SPB0_IO
- net SP2_IO renamed SPB1_IO
- J30 pad 3: +3V3 -> SPB2_IO
- J30 pad 4: +5V_AUX -> SPB3_IO
- J30 pad 5: GND -> SPB4_IO
- R97 pad 1: VLV_SP1 -> MCP_B0
- R98 pad 1: VLV_SP2 -> MCP_B1
- U3 pad 1: CHEM1_MIN -> MCP_B0
- U3 pad 2: CHEM1_MAX -> MCP_B1
- U3 pad 3: CHEM2_MIN -> MCP_B2
- U3 pad 4: CHEM2_MAX -> MCP_B3
- U3 pad 5: CHEM3_MIN -> MCP_B4
- U3 pad 6: CHEM3_MAX -> MCP_B5
Routing:
- net CHEM3_MIN: track 96.4 -> 0.00 mm, vias 3 -> 0
- net CHEM2_MAX: track 91.5 -> 0.00 mm, vias 9 -> 0
- net MCP_B3: track 0.00 -> 69.3 mm, vias 0 -> 2
- net CHEM3_MAX: track 64.8 -> 0.00 mm, vias 6 -> 0
- net VLV_SP2: track 117.2 -> 54.8 mm, vias 9 -> 2
- net C6_TXD: track 100.3 -> 45.2 mm, vias 4 -> 0
- net SNS_C3_MIN: track 55.1 -> 0.00 mm
- net SNS_FLOW: track 67.5 -> 24.0 mm
- net SNS_C3_MAX: track 42.1 -> 0.00 mm, vias 1 -> 0
- net SNS_C2_MIN: track 41.6 -> 0.00 mm, vias 2 -> 0
- net +3V3: track 259.5 -> 301.0 mm, vias 6 -> 7
- net MCP_B5: track 0.00 -> 40.0 mm, vias 0 -> 6
- net MCP_B2: track 0.00 -> 40.0 mm, vias 0 -> 4
- net CHEM2_MIN: track 38.7 -> 0.00 mm, vias 4 -> 0
- net +5V_SENS: track 116.9 -> 79.5 mm, vias 0 -> 1
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Other:
- board text added: "+ 12V OUT 2A -"
- board text added: "+ 5V OUT 1A -"
- board text added: "2026-10-22"
- board text added: "B0"
- board text added: "B1"
- board text added: "B2"
- board text added: "B3"
- board text added: "B4"
- board text added: "B5"
- board text added: "Board v1.2"
- board text added: "FilMachine Board v1.2 - 2026-10-22"
- board text added: "GPIO SPARE (3,3 V)"
- board text removed: "+ a sinistra, - a destra"
- board text removed: "2026-10"
- board text removed: "A6"
- board text removed: "A7"
- board text removed: "Board v1.1"
- board text removed: "CHEM 1"
- board text removed: "CHEM 2"
- board text removed: "CHEM 3"
- board text removed: "FilMachine Board v1.1 - 2026-10"
- board text removed: "GPIO SPARE"
- board text removed: "sx 12V OUT 2A dx 5V OUT 1A"

Commit message: PCB recheck Fable
Parts:
- R80, R82: value 10k -> 4.7k
Other:
- board text added: "+ 12V -"
- board text added: "+ 5V -"
- board text added: "12V IN H1"
- board text added: "12V IN H2"
- board text added: "12V IN MAIN"
- board text added: "12V OUT 2A"
- board text added: "2026-10-23"
- board text added: "5V OUT 1A"
- board text added: "A"
- board text added: "B"
- board text added: "FilMachine Board v1.2 - 2026-10-23"
- board text added: "GPIO SPARE 3V3"
- board text added: "PUMP"
- board text removed: "+ 12V IN HEATER 1 -"
- board text removed: "+ 12V IN HEATER 2 -"
- board text removed: "+ 12V IN MAIN -"
- board text removed: "+ 12V OUT 2A -"
- board text removed: "+ 5V OUT 1A -"
- board text removed: "2026-10-22"
- board text removed: "B PUMP A"
- board text removed: "FilMachine Board v1.2 - 2026-10-22"
- board text removed: "GPIO SPARE (3,3 V)"
