File: PCB/kicad/drives.kicad_sch (KiCad schematic)
At the start: 34 parts, among them J20 PUMP, J21 MOTOR, J22 SERVO, U10 DRV8871DDA, U6 74LVC2G08, U7 74LVC2G08, U8 BTN8982TA, U9 BTN8982TA

Commit message: new board
Parts:
- removed C60: 100uF 10V, Capacitor_SMD:C_1210_3225Metric, symbol Device:C
- removed J20: PUMP, TerminalBlock_Phoenix:TerminalBlock_Phoenix_MKDS-3-2-5.08_1x02_P5.08mm_Horizontal, symbol Connector_Generic:Conn_01x02
- removed J21: MOTOR, TerminalBlock_Phoenix:TerminalBlock_Phoenix_PT-1,5-2-3.5-H_1x02_P3.50mm_Horizontal, symbol Connector_Generic:Conn_01x02
- removed J22: SERVO, Connector_PinHeader_2.54mm:PinHeader_1x03_P2.54mm_Vertical, symbol Connector_Generic:Conn_01x03
- added C56: 470uF 25V, Capacitor_THT:CP_Radial_D10.0mm_P5.00mm, symbol Device:C_Polarized
- added J25: PUMP, FM:TB_WJ500V-5.08-2P, symbol Connector_Generic:Conn_01x02
- added J26: MOTOR, FM:TB_DB301V-3.5-2P, symbol Connector_Generic:Conn_01x02
- added J27: SERVO, Connector_PinHeader_2.54mm:PinHeader_1x03_P2.54mm_Vertical, symbol Connector_Generic:Conn_01x03
- C50, C51: LCSC (none) -> C14663; Manufacturer Samsung/Murata (generic) -> Samsung/Yageo (JLCPCB basic)
- C52, C53, C58: LCSC (none) -> C49678; Manufacturer Samsung/Murata (generic) -> Samsung/Yageo (JLCPCB basic)
- C54, C61: LCSC (none) -> C1588; Manufacturer Samsung/Murata (generic) -> Samsung/Yageo (JLCPCB basic)
- C55: LCSC (none) -> C338188; MPN EEU-FR1E471 -> 25ZLH470MEFC10X12.5; Manufacturer Panasonic -> Rubycon
- C57: footprint Capacitor_SMD:C_1210_3225Metric -> Capacitor_SMD:C_1206_3216Metric; LCSC (none) -> C13585; MPN GRM32ER71H106KA12L -> MLCC 10uF 50V; Manufacturer Samsung/Murata (generic) -> Samsung/Yageo (JLCPCB basic)
- C59: footprint Capacitor_SMD:C_1210_3225Metric -> Capacitor_SMD:C_1206_3216Metric; LCSC (none) -> C12891; MPN GRM32ER71E226KE15L -> MLCC 22uF 25V; Manufacturer Samsung/Murata (generic) -> Samsung/Yageo (JLCPCB basic)
- C60: renamed from C56; value 470uF 25V -> 47uF 10V; footprint Capacitor_THT:CP_Radial_D10.0mm_P5.00mm -> Capacitor_SMD:C_1206_3216Metric; symbol Device:C_Polarized -> Device:C; LCSC (none) -> C96123; MPN EEU-FR1E471 -> MLCC 47uF 10V; Manufacturer Panasonic -> Samsung/Yageo (JLCPCB basic)
- R70, R71, R72, R73, R74, R75, R76: LCSC (none) -> C25803; Manufacturer Yageo/UniOhm (generic) -> UNI-ROYAL
- R80, R82: LCSC (none) -> C25804; Manufacturer Yageo/UniOhm (generic) -> UNI-ROYAL
- R84: value 10k -> 1k; LCSC (none) -> C21190; MPN 0603 10k 1% -> 0603 1k 1%; Manufacturer Yageo/UniOhm (generic) -> UNI-ROYAL
- R85, R88: LCSC (none) -> C22843; Manufacturer Yageo/UniOhm (generic) -> UNI-ROYAL
- R86: LCSC (none) -> C22984; Manufacturer Yageo/UniOhm (generic) -> UNI-ROYAL
- R87: LCSC (none) -> C22962; Manufacturer Yageo/UniOhm (generic) -> UNI-ROYAL
- U10: LCSC (none) -> C75864
- U6, U7: LCSC (none) -> C352973
- U8, U9: value BTN8982TA -> BTN8962TA; LCSC (none) -> C112630; MPN BTN8982TAAUMA1 -> BTN8962TAAUMA1
Connections:
- net +12V_PUMP: now also C56.1; no longer C60.1
- net +5V: now also C60.1, J27.2 (Pin_2)
- net GND: now also C56.2, J27.3 (Pin_3)
- net MOT_OUT_A: now also J26.1 (Pin_1)
- net MOT_OUT_B: now also J26.2 (Pin_2)
- net PUMP_OUT_A: now also J25.1 (Pin_1)
- net PUMP_OUT_B: now also J25.2 (Pin_2)
- net SERVO_SIG: now also J27.1 (Pin_1)

Commit message: new pcb
Parts:
- removed U9: BTN8962TA, Package_TO_SOT_SMD:TO-263-7_TabPin8, symbol Power_Management:BTN8982TA
- added unit 2 of U6
- U9: renamed from U6; value 74LVC2G08 -> BTN8962TA; footprint Package_SO:SSOP-8_2.95x2.8mm_P0.65mm -> Package_TO_SOT_SMD:TO-263-7_TabPin8; symbol 74xGxx:74LVC2G08 -> Power_Management:BTN8982TA; LCSC C352973 -> C112630; MPN SN74LVC2G08DCTR -> BTN8962TAAUMA1; Manufacturer Texas Instruments -> Infineon
Connections:
- net +12V_PUMP: now also U9.7
- net GND: now also U9.1, U9.5 (SR)
- net PUMP_B_CTL: now also U6.3; no longer U9.3
- net PUMP_B_IN: now also U9.2 (IN)
- net PUMP_ENA: now also U6.6; no longer U9.6
- net PUMP_IN2: now also U6.5; no longer U9.5
- net PUMP_INH: now also U9.3 (INH)
- net PUMP_IS_B: now also U9.6 (IS)
- net PUMP_OUT_B: now also U9.4, U9.8

Commit message: PCB recheck Fable
Parts:
- R80, R82: value 10k -> 4.7k; LCSC C25804 -> C23162; MPN 0603 10k 1% -> 0603 4.7k 1%
Changed lines of the file:
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@@
 			(effects (font (size 1.27 1.27)))
 		)
-		(property "Value" "10k"
+		(property "Value" "4.7k"
 			(at 73.66 101.83 0)
 			(effects (font (size 1.27 1.27)))
@@
 			(effects (font (size 1.27 1.27)) (hide yes))
 		)
-		(property "Description" "Serie ingresso IN (datasheet: > 7 kOhm)"
+		(property "Description" "Serie ingresso IN (4,7k: livello alto >= 2,5 V con logica 3,3 V e I_IN(H) max 150 uA)"
 			(at 73.66 96.52 0)
 			(effects (font (size 1.27 1.27)) (hide yes))
 		)
-		(property "MPN" "0603 10k 1%"
+		(property "MPN" "0603 4.7k 1%"
 			(at 73.66 96.52 0)
 			(effects (font (size 1.27 1.27)) (hide yes))
@@
 			(effects (font (size 1.27 1.27)) (hide yes))
 		)
-		(property "LCSC" "C25804"
+		(property "LCSC" "C23162"
 			(at 73.66 96.52 0)
 			(effects (font (size 1.27 1.27)) (hide yes))
@@
 			(effects (font (size 1.27 1.27)))
 		)
-		(property "Value" "10k"
+		(property "Value" "4.7k"
 			(at 142.24 101.83 0)
 			(effects (font (size 1.27 1.27)))
@@
 			(effects (font (size 1.27 1.27)) (hide yes))
 		)
-		(property "Description" "Serie ingresso IN (datasheet: > 7 kOhm)"
+		(property "Description" "Serie ingresso IN (4,7k: livello alto >= 2,5 V con logica 3,3 V e I_IN(H) max 150 uA)"
 			(at 142.24 96.52 0)
 			(effects (font (size 1.27 1.27)) (hide yes))
 		)
-		(property "MPN" "0603 10k 1%"
+		(property "MPN" "0603 4.7k 1%"
 			(at 142.24 96.52 0)
 			(effects (font (size 1.27 1.27)) (hide yes))
@@
 			(effects (font (size 1.27 1.27)) (hide yes))
 		)
-		(property "LCSC" "C25804"
+		(property "LCSC" "C23162"
 			(at 142.24 96.52 0)
 			(effects (font (size 1.27 1.27)) (hide yes))
@@
 			(effects (font (size 1.27 1.27)) (hide yes))
 		)
-		(property "Description" "Pompa Marco UP3-R"
+		(property "Description" "Pompa peristaltica Kamoer KPHM600 (A = pin 1, B = pin 2; qualsiasi motore DC 12 V reversibile)"
 			(at 254 78.74 0)
 			(effects (font (size 1.27 1.27)) (hide yes))
